File: kicad-project/gsmGuard.kicad_pcb (KiCad board)
At the start: 2 copper layers, 70.9 x 45.6 mm, 37 parts, among them J1 Conn_01x02_Female, J2 Conn_01x03_Male, J3 Conn_01x04_Male, Q1 IRLML6401, SW1 SW_Reed, U1 ArduinoProMini, U2 RTC_DS3231, U3 USB_UART, U4 SIM800C, U5 MH-SR602

Commit message: fix resistor values
Parts:
- R10, R11: value 4.7k -> 1k
Changed lines of the file:
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@@
       (effects (font (size 1 1) (thickness 0.15)) (justify mirror))
     )
-    (fp_text value 4.7k (at 0 -1.95 270) (layer B.Fab)
+    (fp_text value 1k (at 0 -1.95 270) (layer B.Fab)
       (effects (font (size 1 1) (thickness 0.15)) (justify mirror))
     )
@@
       (effects (font (size 1 1) (thickness 0.15)) (justify mirror))
     )
-    (fp_text value 4.7k (at 0 -1.95 180) (layer B.Fab)
+    (fp_text value 1k (at 0 -1.95 180) (layer B.Fab)
       (effects (font (size 1 1) (thickness 0.15)) (justify mirror))
     )
