File: kicad-project/gsmGuard.sch (KiCad schematic (older format))
At the start: 37 parts, among them J1 Conn_01x02_Female, J2 Conn_01x03_Male, J3 Conn_01x04_Male, Q1 IRLML6401, SW1 SW_Reed, U1 ArduinoProMini, U2 RTC_DS3231, U3 USB_UART, U4 SIM800C, U5 MH-SR602

Commit message: fix resistor values
Parts:
- R10, R11: value 4.7k -> 1k
Changed lines of the file:
@@
 LIBS:contrib
 LIBS:valves
-LIBS:gsmGuard-cache
 EELAYER 26 0
 EELAYER END
@@
 P 5050 1750
 F 0 "R10" H 5120 1796 50  0000 L CNN
-F 1 "4.7k" H 5120 1705 50  0000 L CNN
+F 1 "1k" H 5120 1705 50  0000 L CNN
 F 2 "Resistors_SMD:R_1206" V 4980 1750 50  0001 C CNN
 F 3 "~" H 5050 1750 50  0001 C CNN
@@
 P 4700 2700
 F 0 "R11" H 4770 2746 50  0000 L CNN
-F 1 "4.7k" H 4770 2655 50  0000 L CNN
+F 1 "1k" H 4770 2655 50  0000 L CNN
 F 2 "Resistors_SMD:R_1206" V 4630 2700 50  0001 C CNN
 F 3 "~" H 4700 2700 50  0001 C CNN
